Commit message: updated

File: rover_project/urdf/rover.urdf (robot description, URDF)
Before this commit: robot rover, 9 links, 8 joints
Joints:
- joint base_footprint_joint: origin xyz=0 0 0.03 rpy=0 0 0 -> xyz=0 0 0 rpy=0 0 0
- joint front_left_wheel_joint: axis 0 0 1 -> 0 1 0; origin xyz=0.2 -0.14 -0.06 rpy=1.570796 0 0 -> xyz=0.15 0.175 -0.03 rpy=0 0 0
- joint front_right_wheel_joint: axis 0 0 1 -> 0 1 0; origin xyz=0.2 0.14 -0.06 rpy=1.570796 0 0 -> xyz=0.15 -0.175 -0.03 rpy=0 0 0
- joint rear_left_wheel_joint: axis 0 0 1 -> 0 1 0; mimic joint=front_left_wheel_joint multiplier=1 offset=0 -> (none); origin xyz=-0.2 0.14 -0.06 rpy=1.570796 0 0 -> xyz=-0.15 0.175 -0.03 rpy=0 0 0
- joint rear_right_wheel_joint: axis 0 0 1 -> 0 1 0; mimic joint=front_right_wheel_joint multiplier=1 offset=0 -> (none); origin xyz=-0.2 -0.14 -0.06 rpy=1.570796 0 0 -> xyz=-0.15 -0.175 -0.03 rpy=0 0 0

Commit message: improved urdf
Updated material definitions, added new mounts for sensors, and modified joint configurations for the rover model. Adjusted inertial properties and added ROS2 control configuration.

File: rover_project/urdf/rover.urdf (robot description, URDF)
Before this commit: robot rover, 9 links, 8 joints
Links:
- removed link camera_link
- removed link camera_mount
- removed link laser_link
- added link laser_link1, mass 0.1; collision cylinder length=0.05 radius=0.05; visual cylinder length=0.05 radius=0.05
- added link laser_link2, mass 0.1; collision cylinder length=0.05 radius=0.05; visual cylinder length=0.05 radius=0.05
- added link link1_mount, mass 0.1; visual box size=0.08 0.04 0.04
- added link link2_mount, mass 0.1; visual box size=0.08 0.04 0.04
Joints:
- removed joint camera_joint
- removed joint camera_link_joint
- removed joint laser_joint
- added joint base_to_link1_joint: type fixed, parent base_link, child link1_mount, origin xyz=0 0 0.05 rpy=0 0 0
- added joint base_to_link2_joint: type fixed, parent base_link, child link2_mount, origin xyz=0.20 0 0.09 rpy=0 0 0
- added joint laser_joint1: type fixed, parent link1_mount, child laser_link1, origin xyz=0 0 0.064 rpy=1.570796 0 0
- added joint laser_joint2: type fixed, parent link2_mount, child laser_link2, origin xyz=0 0 0.03 rpy=0 0 0
- joint base_footprint_joint: origin xyz=0 0 0 rpy=0 0 0 -> xyz=0 0 0.05 rpy=0 0 0
- joint front_left_wheel_joint: axis 0 1 0 -> 0 0 1; origin xyz=0.15 0.175 -0.03 rpy=0 0 0 -> xyz=0.15 0.175 0.03 rpy=${-pi/2} 0 0
- joint front_right_wheel_joint: axis 0 1 0 -> 0 0 -1; origin xyz=0.15 -0.175 -0.03 rpy=0 0 0 -> xyz=0.15 -0.175 0.03 rpy=${pi/2} 0 0
- joint rear_left_wheel_joint: axis 0 1 0 -> 0 0 1; origin xyz=-0.15 0.175 -0.03 rpy=0 0 0 -> xyz=-0.15 0.175 0.03 rpy=${-pi/2} 0 0
- joint rear_right_wheel_joint: axis 0 1 0 -> 0 0 -1; origin xyz=-0.15 -0.175 -0.03 rpy=0 0 0 -> xyz=-0.15 -0.175 0.03 rpy=${pi/2} 0 0
